File: controller/pcb/Greenhouse Board.kicad_sch (KiCad schematic)
At the start: 30 parts, among them J1 12V, J2 window control, J3 fan control, J4 misting control, J5 light_sensor, J6 GND, J7 T+H sensor, J8 temp sensor 1, J9 temp sensor 2, Q1 DMN53D0LW-7, Q2 DMN53D0LW-7, Q3 DMN6140LQ-7, U1 XAIO ESP32-C3, U2 12-5V DC/DC

Commit message: Commit most recent schematic changes
Parts:
- added R7: 10k, Resistor_SMD:R_0805_2012Metric_Pad1.20x1.40mm_HandSolder, symbol Device:R_US
Other:
- moved on the sheet: C3, R9
Changed lines of the file:
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@@
 	)
 	(junction
-		(at 158.75 152.4)
+		(at 175.26 152.4)
 		(diameter 0)
 		(color 0 0 0 0)
@@
 	)
 	(junction
-		(at 158.75 129.54)
+		(at 175.26 129.54)
 		(diameter 0)
 		(color 0 0 0 0)
@@
 	)
 	(junction
-		(at 140.97 139.7)
+		(at 135.89 139.7)
 		(diameter 0)
 		(color 0 0 0 0)
@@
 	)
 	(junction
-		(at 195.58 92.71)
+		(at 135.89 129.54)
 		(diameter 0)
 		(color 0 0 0 0)
 	)
 	(junction
-		(at 100.33 82.55)
+		(at 195.58 92.71)
 		(diameter 0)
 		(color 0 0 0 0)
 	)
 	(junction
-		(at 140.97 129.54)
+		(at 100.33 82.55)
 		(diameter 0)
 		(color 0 0 0 0)
@@
 	(wire
 		(pts
-			(xy 158.75 144.78) (xy 158.75 152.4)
+			(xy 175.26 144.78) (xy 175.26 152.4)
 		)
 		(stroke
@@
 	(wire
 		(pts
-			(xy 140.97 129.54) (xy 140.97 130.81)
-		)
-		(stroke
-			(width 0)
-			(type default)
-		)
-	)
-	(wire
-		(pts
-			(xy 130.81 152.4) (xy 158.75 152.4)
+			(xy 135.89 129.54) (xy 135.89 130.81)
 		)
 		(stroke
@@
 	(wire
 		(pts
-			(xy 130.81 142.24) (xy 133.35 142.24)
+			(xy 130.81 142.24) (xy 156.21 142.24)
 		)
 		(stroke
@@
 	(wire
 		(pts
+			(xy 135.89 129.54) (xy 175.26 129.54)
+		)
+		(stroke
+			(width 0)
+			(type default)
+		)
+	)
+	(wire
+		(pts
+			(xy 130.81 152.4) (xy 175.26 152.4)
+		)
+		(stroke
+			(width 0)
+			(type default)
+		)
+	)
+	(wire
+		(pts
 			(xy 177.8 64.77) (xy 177.8 67.31)
 		)
@@
 	(wire
 		(pts
-			(xy 130.81 129.54) (xy 140.97 129.54)
+			(xy 130.81 129.54) (xy 135.89 129.54)
 		)
 		(stroke
@@
 	(wire
 		(pts
-			(xy 158.75 121.92) (xy 158.75 129.54)
+			(xy 175.26 121.92) (xy 175.26 129.54)
+		)
+		(stroke
+			(width 0)
+			(type default)
+		)
+	)
+	(wire
+		(pts
+			(xy 135.89 139.7) (xy 139.7 139.7)
 		)
 		(stroke
@@
 	(wire
 		(pts
-			(xy 130.81 139.7) (xy 140.97 139.7)
+			(xy 130.81 139.7) (xy 135.89 139.7)
 		)
 		(stroke
@@
 	(wire
 		(pts
-			(xy 158.75 152.4) (xy 158.75 156.21)
+			(xy 175.26 152.4) (xy 175.26 156.21)
 		)
 		(stroke
@@
 	(wire
 		(pts
-			(xy 158.75 129.54) (xy 158.75 137.16)
+			(xy 175.26 129.54) (xy 175.26 137.16)
 		)
 		(stroke
@@
 	(wire
 		(pts
-			(xy 140.97 138.43) (xy 140.97 139.7)
+			(xy 135.89 138.43) (xy 135.89 139.7)
 		)
 		(stroke
@@
 	(wire
 		(pts
-			(xy 140.97 139.7) (xy 147.32 139.7)
-		)
-		(stroke
-			(width 0)
-			(type default)
-		)
-	)
-	(wire
-		(pts
 			(xy 29.21 36.83) (xy 44.45 36.83)
 		)
@@
 	(wire
 		(pts
-			(xy 140.97 129.54) (xy 158.75 129.54)
-		)
-		(stroke
-			(width 0)
-			(type default)
-		)
-	)
-	(wire
-		(pts
 			(xy 207.01 146.05) (xy 207.01 148.59)
 		)
@@
 	)
 	(label "temp_bus"
-		(at 147.32 139.7 0)
+		(at 139.7 139.7 0)
 		(effects
 			(font
@@
 	)
 	(label "DHT22_Sensor"
-		(at 133.35 142.24 0)
+		(at 156.21 142.24 0)
 		(effects
 			(font
@@
 	(symbol
 		(lib_id "Device:R_US")
-		(at 140.97 134.62 0)
+		(at 135.89 134.62 0)
 		(unit 1)
 		(exclude_from_sim no)
@@
 		(fields_autoplaced yes)
 		(property "Reference" "R9"
-			(at 143.51 133.3499 0)
+			(at 138.43 133.3499 0)
 			(effects
 				(font
@@
 		)
 		(property "Value" "4.7k"
-			(at 143.51 135.8899 0)
+			(at 138.43 135.8899 0)
 			(effects
 				(font
@@
 		)
 		(property "Footprint" "Resistor_SMD:R_0805_2012Metric_Pad1.20x1.40mm_HandSolder"
-			(at 141.986 134.874 90)
+			(at 136.906 134.874 90)
 			(effects
 				(font
@@
 		)
 		(property "Datasheet" "~"
-			(at 140.97 134.62 0)
+			(at 135.89 134.62 0)
 			(effects
 				(font
@@
 		)
 		(property "Description" "Resistor, US symbol"
-			(at 140.97 134.62 0)
+			(at 135.89 134.62 0)
 			(effects
 				(font
@@
 	(symbol
 		(lib_id "Device:R_US")
+		(at 152.4 135.89 0)
+		(unit 1)
+		(exclude_from_sim no)
+		(in_bom yes)
+		(on_board yes)
+		(dnp no)
+		(fields_autoplaced yes)
+		(property "Reference" "R7"
+			(at 154.94 134.6199 0)
+			(effects
+				(font
+					(size 1.27 1.27)
+				)
+				(justify left)
+			)
+		)
+		(property "Value" "10k"
+			(at 154.94 137.1599 0)
+			(effects
+				(font
+					(size 1.27 1.27)
+				)
+				(justify left)
+			)
+		)
+		(property "Footprint" "Resistor_SMD:R_0805_2012Metric_Pad1.20x1.40mm_HandSolder"
+			(at 153.416 136.144 90)
+			(effects
+				(font
+					(size 1.27 1.27)
+				)
+				(hide yes)
+			)
+		)
+		(property "Datasheet" "~"
+			(at 152.4 135.89 0)
+			(effects
+				(font
+					(size 1.27 1.27)
+				)
+				(hide yes)
+			)
+		)
+		(property "Description" "Resistor, US symbol"
+			(at 152.4 135.89 0)
+			(effects
+				(font
+					(size 1.27 1.27)
+				)
+				(hide yes)
+			)
+		)
+		(pin "2"
+		)
+		(pin "1"
+		)
+		(instances
+			(project "Greenhouse Board"
+				(path "/c4158e2f-5e89-4df3-97ea-8a8d31d33e4c"
+					(reference "R7")
+					(unit 1)
+				)
+			)
+		)
+	)
+	(symbol
+		(lib_id "Device:R_US")
 		(at 207.01 152.4 0)
 		(unit 1)
@@
 	(symbol
 		(lib_id "Device:C")
-		(at 158.75 140.97 0)
+		(at 175.26 140.97 0)
 		(unit 1)
 		(exclude_from_sim no)
@@
 		(fields_autoplaced yes)
 		(property "Reference" "C3"
-			(at 162.56 139.6999 0)
+			(at 179.07 139.6999 0)
 			(effects
 				(font
@@
 		)
 		(property "Value" ".1u"
-			(at 162.56 142.2399 0)
+			(at 179.07 142.2399 0)
 			(effects
 				(font
@@
 		)
 		(property "Footprint" "Capacitor_SMD:C_0805_2012Metric"
-			(at 159.7152 144.78 0)
+			(at 176.2252 144.78 0)
 			(effects
 				(font
@@
 		)
 		(property "Datasheet" "~"
-			(at 158.75 140.97 0)
+			(at 175.26 140.97 0)
 			(effects
 				(font
@@
 		)
 		(property "Description" "Unpolarized capacitor"
-			(at 158.75 140.97 0)
+			(at 175.26 140.97 0)
 			(effects
 				(font
@@
 	(symbol
 		(lib_id "power:GND")
-		(at 158.75 156.21 0)
+		(at 175.26 156.21 0)
 		(unit 1)
 		(exclude_from_sim no)
@@
 		(fields_autoplaced yes)
 		(property "Reference" "#PWR04"
-			(at 158.75 162.56 0)
+			(at 175.26 162.56 0)
 			(effects
 				(font
@@
 		)
 		(property "Value" "GND"
-			(at 158.75 161.29 0)
+			(at 175.26 161.29 0)
 			(effects
 				(font
@@
 		)
 		(property "Footprint" ""
-			(at 158.75 156.21 0)
+			(at 175.26 156.21 0)
 			(effects
 				(font
@@
 		)
 		(property "Datasheet" ""
-			(at 158.75 156.21 0)
+			(at 175.26 156.21 0)
 			(effects
 				(font
@@
 		)
 		(property "Description" "Power symbol creates a global label with name \"GND\" , ground"
-			(at 158.75 156.21 0)
+			(at 175.26 156.21 0)
 			(effects
 				(font
@@
 	(symbol
 		(lib_id "power:+5V")
-		(at 158.75 121.92 0)
+		(at 175.26 121.92 0)
 		(unit 1)
 		(exclude_from_sim no)
@@
 		(fields_autoplaced yes)
 		(property "Reference" "#PWR08"
-			(at 158.75 125.73 0)
+			(at 175.26 125.73 0)
 			(effects
 				(font
@@
 		)
 		(property "Value" "+5V"
-			(at 158.75 116.84 0)
+			(at 175.26 116.84 0)
 			(effects
 				(font
@@
 		)
 		(property "Footprint" ""
-			(at 158.75 121.92 0)
+			(at 175.26 121.92 0)
 			(effects
 				(font
@@
 		)
 		(property "Datasheet" ""
-			(at 158.75 121.92 0)
+			(at 175.26 121.92 0)
 			(effects
 				(font
@@
 		)
 		(property "Description" "Power symbol creates a global label with name \"+5V\""
-			(at 158.75 121.92 0)
+			(at 175.26 121.92 0)
 			(effects
 				(font
